File: matrix_io_board.brd (EAGLE design)
At the start: 155.7 x 39.1 mm, 101 parts, among them IC1 6N138, IC2 LM27675M5_CHARGEPUMP, IC3 LM324D, IC4 MCP4728_QUAD_DAC, IC5 4504D, IC6 74AHC1G14DBV, IC7 FDS8958B, IC8 SP34063A_BOOST_REG

Commit message: rename
Parts:
- GD2: value GD -> (none)
- renumbered 5V1 to 5V., GND26 to GD1, GND38 to GD2
Changed lines of the file:
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@@
 <text x="63.881" y="8.5725" size="1.27" layer="21" font="vector" ratio="20" rot="R270">10V</text>
 <text x="66.548" y="10.922" size="1.27" layer="21" font="vector" ratio="20">VIN</text>
-<text x="46.736" y="31.369" size="1.778" layer="21" font="vector" rot="R270">hotchk155</text>
+<text x="46.736" y="31.369" size="1.778" layer="21" font="vector" ratio="20" rot="R270">hotchk155</text>
 <wire x1="58.2295" y1="38.0365" x2="50.8" y2="38.0365" width="0.254" layer="21"/>
 <wire x1="50.8" y1="38.0365" x2="50.8" y2="35.3695" width="0.254" layer="21"/>
@@
 <wire x1="70.612" y1="5.6515" x2="70.612" y2="8.1915" width="0.254" layer="21"/>
 <wire x1="70.612" y1="8.1915" x2="65.5955" y2="8.1915" width="0.254" layer="21"/>
-<text x="86.6775" y="28.6385" size="1.778" layer="52" font="vector" rot="MR180">matrix synth i/o board rev 1</text>
+<text x="86.6775" y="28.6385" size="1.778" layer="52" font="vector" ratio="20" rot="MR180">matrix synth i/o board rev 1</text>
 </plain>
 <attributes>
@@
 </element>
 <element name="5V" library="pinhead" package="1X01" value="" x="105.41" y="1.27" smashed="yes">
-<attribute name="NAME" x="106.1212" y="-7.6962" size="1.27" layer="25" font="vector" ratio="20" rot="R90"/>
+<attribute name="NAME" x="104.7877" y="2.8448" size="1.27" layer="26" font="vector" ratio="20" rot="MR90"/>
 <attribute name="VALUE" x="104.14" y="-1.905" size="1.27" layer="27"/>
 </element>
 <element name="GND" library="pinhead" package="1X01" value="" x="148.59" y="1.27" smashed="yes">
-<attribute name="NAME" x="148.9202" y="-7.7597" size="1.27" layer="25" font="vector" ratio="20" rot="R90"/>
+<attribute name="NAME" x="148.0312" y="2.8448" size="1.27" layer="26" font="vector" ratio="20" rot="MR90"/>
 <attribute name="VALUE" x="147.32" y="-1.905" size="1.27" layer="27"/>
 </element>
@@
 <attribute name="VALUE" x="134.874" y="32.004" size="1.27" layer="27" rot="R180"/>
 </element>
-<element name="GND38" library="pinhead" package="1X01" value="GD" x="110.49" y="1.27" smashed="yes" rot="R90">
-<attribute name="VALUE" x="111.3155" y="-7.62" size="1.27" layer="27" font="vector" ratio="20" rot="R90"/>
+<element name="GD2" library="pinhead" package="1X01" value="" x="110.49" y="1.27" smashed="yes" rot="R90">
+<attribute name="NAME" x="110.8202" y="2.7813" size="1.27" layer="26" font="vector" ratio="20" rot="MR90"/>
 </element>
 <element name="L1" library="SparkFun" package="1210" value="" x="108.6485" y="12.1285" smashed="yes" rot="R180">
@@
 </element>
 <element name="SCL" library="pinhead" package="1X01" value="" x="133.35" y="1.27" smashed="yes" rot="R90">
-<attribute name="NAME" x="134.0612" y="-7.6962" size="1.27" layer="25" font="vector" ratio="20" rot="R90"/>
+<attribute name="NAME" x="132.9182" y="2.5908" size="1.27" layer="26" font="vector" ratio="20" rot="MR90"/>
 <attribute name="VALUE" x="136.525" y="0" size="1.27" layer="27" rot="R90"/>
 </element>
 <element name="SDA" library="pinhead" package="1X01" value="" x="135.89" y="1.27" smashed="yes" rot="R90">
-<attribute name="NAME" x="136.6012" y="-7.6962" size="1.27" layer="25" font="vector" ratio="20" rot="R90"/>
+<attribute name="NAME" x="135.3312" y="2.5273" size="1.27" layer="26" font="vector" ratio="20" rot="MR90"/>
 <attribute name="VALUE" x="139.065" y="0" size="1.27" layer="27" rot="R90"/>
 </element>
 <element name="G3" library="pinhead" package="1X01" value="" x="130.81" y="1.27" smashed="yes" rot="R90">
-<attribute name="NAME" x="131.5212" y="-7.6962" size="1.27" layer="25" font="vector" ratio="20" rot="R90"/>
+<attribute name="NAME" x="130.3147" y="2.6543" size="1.27" layer="26" font="vector" ratio="20" rot="MR90"/>
 <attribute name="VALUE" x="133.985" y="0" size="1.27" layer="27" rot="R90"/>
 </element>
 <element name="G2" library="pinhead" package="1X01" value="" x="128.27" y="1.27" smashed="yes" rot="R90">
-<attribute name="NAME" x="128.9812" y="-7.6962" size="1.27" layer="25" font="vector" ratio="20" rot="R90"/>
+<attribute name="NAME" x="127.7747" y="2.7178" size="1.27" layer="26" font="vector" ratio="20" rot="MR90"/>
 <attribute name="VALUE" x="131.445" y="0" size="1.27" layer="27" rot="R90"/>
 </element>
 <element name="G1" library="pinhead" package="1X01" value="" x="123.19" y="1.27" smashed="yes" rot="R90">
-<attribute name="NAME" x="123.9012" y="-7.6962" size="1.27" layer="25" font="vector" ratio="20" rot="R90"/>
+<attribute name="NAME" x="122.8217" y="2.7813" size="1.27" layer="26" font="vector" ratio="20" rot="MR90"/>
 <attribute name="VALUE" x="126.365" y="0" size="1.27" layer="27" rot="R90"/>
 </element>
 <element name="CKOUT" library="pinhead" package="1X01" value="" x="146.05" y="1.27" smashed="yes" rot="R90">
-<attribute name="NAME" x="146.6342" y="-7.6962" size="1.27" layer="25" font="vector" ratio="20" rot="R90"/>
+<attribute name="NAME" x="145.6817" y="2.7178" size="1.27" layer="26" font="vector" ratio="20" rot="MR90"/>
 <attribute name="VALUE" x="149.225" y="0" size="1.27" layer="27" rot="R90"/>
 </element>
 <element name="GX" library="pinhead" package="1X01" value="" x="120.65" y="1.27" smashed="yes" rot="R90">
-<attribute name="NAME" x="121.3612" y="-7.6962" size="1.27" layer="25" font="vector" ratio="20" rot="R90"/>
+<attribute name="NAME" x="120.2182" y="2.7178" size="1.27" layer="26" font="vector" ratio="20" rot="MR90"/>
 <attribute name="VALUE" x="123.825" y="0" size="1.27" layer="27" rot="R90"/>
 </element>
 <element name="G4" library="pinhead" package="1X01" value="" x="125.73" y="1.27" smashed="yes" rot="R90">
-<attribute name="NAME" x="126.4412" y="-7.6962" size="1.27" layer="25" font="vector" ratio="20" rot="R90"/>
+<attribute name="NAME" x="125.2982" y="2.7178" size="1.27" layer="26" font="vector" ratio="20" rot="MR90"/>
 <attribute name="VALUE" x="128.905" y="0" size="1.27" layer="27" rot="R90"/>
 </element>
 <element name="CLKIN" library="pinhead" package="1X01" value="" x="138.43" y="1.27" smashed="yes" rot="R90">
-<attribute name="NAME" x="139.1412" y="-7.6962" size="1.27" layer="25" font="vector" ratio="20" rot="R90"/>
+<attribute name="NAME" x="137.9982" y="2.6543" size="1.27" layer="26" font="vector" ratio="20" rot="MR90"/>
 <attribute name="VALUE" x="141.605" y="0" size="1.27" layer="27" rot="R90"/>
 </element>
 <element name="TX" library="pinhead" package="1X01" value="" x="118.11" y="1.27" smashed="yes" rot="R90">
-<attribute name="NAME" x="118.8212" y="-7.6962" size="1.27" layer="25" font="vector" ratio="20" rot="R90"/>
+<attribute name="NAME" x="117.6147" y="2.7178" size="1.27" layer="26" font="vector" ratio="20" rot="MR90"/>
 <attribute name="VALUE" x="121.285" y="0" size="1.27" layer="27" rot="R90"/>
 </element>
 <element name="RX" library="pinhead" package="1X01" value="" x="115.57" y="1.27" smashed="yes" rot="R90">
-<attribute name="NAME" x="116.2812" y="-7.6962" size="1.27" layer="25" font="vector" ratio="20" rot="R90"/>
+<attribute name="NAME" x="115.2017" y="2.7813" size="1.27" layer="26" font="vector" ratio="20" rot="MR90"/>
 <attribute name="VALUE" x="118.745" y="0" size="1.27" layer="27" rot="R90"/>
 </element>
 <element name="PWRCTL" library="pinhead" package="1X01" value="" x="140.97" y="1.27" smashed="yes" rot="R90">
-<attribute name="NAME" x="141.6812" y="-7.6962" size="1.27" layer="25" font="vector" ratio="20" rot="R90"/>
+<attribute name="NAME" x="141.4907" y="4.6863" size="1.27" layer="26" font="vector" ratio="20" rot="MR90"/>
 <attribute name="VALUE" x="144.145" y="0" size="1.27" layer="27" rot="R90"/>
 </element>
@@
 <attribute name="VALUE" x="92.964" y="1.5875" size="1.27" layer="27"/>
 </element>
-<element name="GND26" library="pinhead" package="1X01" value="GD" x="113.03" y="1.27" smashed="yes">
-<attribute name="VALUE" x="113.665" y="-7.62" size="1.27" layer="27" font="vector" ratio="20" rot="R90"/>
-</element>
-<element name="5V1" library="pinhead" package="1X01" value="" x="107.95" y="1.27" smashed="yes">
-<attribute name="NAME" x="108.6612" y="-7.6962" size="1.27" layer="25" font="vector" ratio="20" rot="R90"/>
+<element name="GD1" library="pinhead" package="1X01" value="GD" x="113.03" y="1.27" smashed="yes">
+<attribute name="NAME" x="112.5728" y="2.8067" size="1.27" layer="26" font="vector" ratio="20" rot="MR90"/>
+</element>
+<element name="5V." library="pinhead" package="1X01" value="" x="107.95" y="1.27" smashed="yes">
+<attribute name="NAME" x="107.3277" y="2.7813" size="1.27" layer="26" font="vector" ratio="20" rot="MR90"/>
 <attribute name="VALUE" x="106.68" y="-1.905" size="1.27" layer="27"/>
 </element>
 <element name="OFFSW" library="pinhead" package="1X01" value="" x="143.51" y="1.27" smashed="yes">
-<attribute name="NAME" x="144.2212" y="-7.6962" size="1.27" layer="25" font="vector" ratio="20" rot="R90"/>
+<attribute name="NAME" x="143.0147" y="2.6543" size="1.27" layer="26" font="vector" ratio="20" rot="MR90"/>
 <attribute name="VALUE" x="142.24" y="-1.905" size="1.27" layer="27"/>
 </element>
@@
 <contactref element="R26" pad="1"/>
 <contactref element="GND" pad="1"/>
-<contactref element="GND38" pad="1"/>
+<contactref element="GD2" pad="1"/>
 <contactref element="C13" pad="-"/>
 <contactref element="MIDI_OUT" pad="2"/>
@@
 <contactref element="D4" pad="C"/>
 <via x="57.15" y="10.287" extent="1-16" drill="0.6"/>
-<contactref element="GND26" pad="1"/>
+<contactref element="GD1" pad="1"/>
 <polygon width="0.8128" layer="16">
 <vertex x="-3.81" y="44.45"/>
@@
 <wire x1="30.099" y1="9.84" x2="30.099" y2="10.033" width="0.6096" layer="1"/>
 <wire x1="30.099" y1="10.033" x2="30.226" y2="10.16" width="0.6096" layer="1"/>
-<contactref element="5V1" pad="1"/>
+<contactref element="5V." pad="1"/>
 <wire x1="98.552" y1="7.554" x2="100.4285" y2="7.554" width="0.3048" layer="1"/>
 <wire x1="100.4285" y1="7.554" x2="100.5865" y2="7.396" width="0.3048" layer="1"/>

Commit message: changes for rev2
Parts:
- removed AUX: (no value), microbuilder:TESTPOINT_ROUND_2MM
- removed GATE: (no value), pinhead:2X03
- removed R23: (no value), rcl:R0805
- added C17, C18, C19, C20, C21: 100n, rcl:C0805
- added R32: 470k, rcl:R0805
- C1, C2, C3: value (none) -> 10u
- C10, C11, C12, C8: value (none) -> 100n
- C15: value (none) -> 470p
- C6: value (none) -> 20p
- R1, R3, R5: value (none) -> 220
- R10, R11, R12, R13, R18, R19, R20, R21, R22, R24, R27, R28, R30: value (none) -> 1k
- R14, R15, R16, R17, R6, R7, R8, R9: value (none) -> 10k/0.1%
- R2, R4: value (none) -> 1k8
- R25, R26: value (none) -> 10k
- R29: value (none) -> 0r33
- R31: value (none) -> 3k
- moved BATT+ 4.60 mm to (154.7, 30.9)
- moved C13 1.27 mm to (109.7, 6.73)
- moved L1 1.27 mm to (109.9, 12.1)
- moved R22 1.02 mm to (91.8, 5.40)
- moved BATT- 0.92 mm to (152.8, 29.0)
- moved C11 0.89 mm to (91.8, 7.81)
- moved R21 0.70 mm to (91.8, 10.3)
- moved R18 0.06 mm to (77.6, 8.64)
- moved R19 0.06 mm to (77.6, 6.35)
- moved R20 0.06 mm to (77.6, 4.06)
Connections:
- removed net N$42: IC5.10, R23.1
- removed net N$50: AUX.P$1, R23.2
- removed net N$71: BATT-.1, U$1.NC
- removed net VGATE: C10.2, GATE.1, GATE.3, GATE.5, IC5.16
- new net N$16: BATT+.1, U$1.NC
- net +10V: now also C10.2, IC5.16; no longer GATE.4
- net +5V: no longer GATE.2
- net +9V: no longer GATE.6
- net GND: now also BATT-.1, C17.1, C18.1, C19.1, C20.1, C21.1, R32.1, U$1.PIN; no longer U$1.BARREL
- net N$36: now also U$1.BARREL; no longer BATT+.1, U$1.PIN
- net N$44: now also C17.2
- net N$45: now also C18.2
- net N$46: now also C19.2
- net N$47: now also C20.2
- net N$48: now also C21.2
- net N$54: now also R32.2
Routing:
- net +10V: track 37.7 -> 72.0 mm, vias 1 -> 3
- net VGATE: track 29.4 -> 0.00 mm, vias 1 -> 0
- net N$71: track 13.5 -> 0.00 mm
- net N$16: track 0.00 -> 13.3 mm
- net +9V: track 163.9 -> 158.4 mm
- net N$36: track 13.5 -> 8.74 mm
- net N$47: track 31.5 -> 35.9 mm
- net N$54: track 24.9 -> 28.5 mm
- net N$42: track 3.47 -> 0.00 mm
- net N$44: track 64.8 -> 67.9 mm, vias 0 -> 2
- net N$46: track 53.6 -> 56.7 mm, vias 0 -> 2
- net N$45: track 62.0 -> 64.8 mm, vias 0 -> 2
- net N$50: track 2.73 -> 0.00 mm
- net +5V: track 229.5 -> 227.1 mm
- net N$48: track 10.6 -> 12.7 mm
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Other:
- board text removed: "10V"
- board text removed: "5V"
- board text removed: "VIN"

Commit message: version 2 ready for fab
Other:
- board text added: "matrix synth i/o board rev 2"
- board text removed: "matrix synth i/o board rev 1"
Changed lines of the file:
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@@
 <wire x1="100.457" y1="13.716" x2="93.6625" y2="13.716" width="0.254" layer="21"/>
 <wire x1="93.6625" y1="13.716" x2="93.6625" y2="12.319" width="0.254" layer="21"/>
-<text x="86.6775" y="28.6385" size="1.778" layer="52" font="vector" ratio="20" rot="MR180">matrix synth i/o board rev 1</text>
+<text x="86.6775" y="28.6385" size="1.778" layer="52" font="vector" ratio="20" rot="MR180">matrix synth i/o board rev 2</text>
 </plain>
 <attributes>
@@
 <wire x1="83.566" y1="6.858" x2="81.5721" y2="6.858" width="0.3048" layer="1"/>
 <wire x1="81.5721" y1="6.858" x2="81.5086" y2="6.9215" width="0.3048" layer="1"/>
-<wire x1="82.169" y1="6.858" x2="81.915" y2="7.112" width="0.3048" layer="16"/>
 <wire x1="128.27" y1="1.27" x2="128.27" y2="10.795" width="0.3048" layer="16"/>
 <wire x1="128.27" y1="10.795" x2="123.952" y2="15.113" width="0.3048" layer="16"/>
@@
 <wire x1="89.408" y1="6.858" x2="83.566" y2="6.858" width="0.3048" layer="16"/>
 <wire x1="89.789" y1="7.239" x2="89.408" y2="6.858" width="0.3048" layer="16"/>
-<wire x1="81.5721" y1="6.858" x2="81.915" y2="7.112" width="0" layer="19" extent="1-16"/>
 </signal>
 <signal name="GATE3">
