File: matrix_io_board.brd (EAGLE design)
At the start: 155.7 x 39.1 mm, 104 parts, among them IC1 6N138, IC2 LM27675M5_CHARGEPUMP, IC3 LM324D, IC4 MCP4728_QUAD_DAC, IC5 4504D, IC6 74AHC1G14DBV, IC7 FDS8958B, IC8 SP34063A_BOOST_REG

Commit message: work in progress
Parts:
- removed CKIN: VERTICAL_3_5MM_SOCKET, jason_eagle6:VERTICAL_3_5MM_SOCKET
- removed GND, GX: (no value), pinhead:1X01
- removed IC6: 74AHC1G14DBV, 74xx-little-de:SOT23-5
- removed MIDI_IN, MIDI_OUT: DIN5PIN, jason_eagle6:EDGEDIN
- added C22: 100n, rcl:C0805
- added CKI, RSI, RSO: WQP-PJ301M-12_JACK, thonkiconn:WQP-PJ301M-12_JACK
- added D7, D8: 0805DIODE, jasons_stuff:0805DIODE
- added GD3, GD4, RSIN, RSOUT: (no value), pinhead:1X01
- added MIDIIN, MIDIOUT: VERTICAL_3_5MM_SOCKETTHONK, jason_eagle6:PJ301CM
- added R23, R33: 1k, rcl:R0805
- added R34: 470k, rcl:R0805
- added U$2: SN74LVC2G14, jason_eagle6:DBV_R-PDSO-G6
- CKO, CVA, CVB, CVC, CVD, GT1, GT2, GT3, GT4: value VERTICAL_3_5MM_SOCKET -> WQP-PJ301M-12_JACK; device jason_eagle6:VERTICAL_3_5MM_SOCKET -> thonkiconn:WQP-PJ301M-12_JACK
- GD1: value GD -> (none)
- L2: device inductors:DR1030 -> jason_eagle6:DR1030
- moved CKO 98.3 mm to (26.7, 21.6), turned to 270 degrees
- moved R32 78.7 mm to (26.7, 11.4), turned to 270 degrees
- moved R24 71.2 mm to (29.2, 11.4), turned to 270 degrees
- moved D4 71.1 mm to (31.8, 11.4), turned to 270 degrees
- moved D3 63.8 mm to (34.3, 11.4)
- moved C12 60.5 mm to (38.1, 5.08), turned to 180 degrees
- moved D5 42.4 mm to (90.6, 6.73)
- moved C14 35.7 mm to (81.0, 5.33), turned to 180 degrees
- moved C11 33.2 mm to (59.8, 16.5)
- moved R31 32.1 mm to (113.0, 3.81), turned to 0 degrees
- moved C13 29.3 mm to (81.0, 12.8), turned to 180 degrees
- moved R30 28.9 mm to (116.6, 3.81), turned to 270 degrees
- moved R28 28.8 mm to (114.9, 13.1)
- moved R29 28.6 mm to (116.6, 8.38), turned to 90 degrees
- moved C15 28.5 mm to (108.2, 3.81)
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Connections:
- removed net CLKIN: CLKIN.1, IC6.4
- new net N$19: IC5.10, R23.1
- new net N$23: CLKIN.1, U$2.6
- new net N$24: R33.2, R34.2, RSI.P$1
- new net N$25: RSIN.1, U$2.4
- new net N$26: D7.C, D8.A, R33.1, U$2.3
- new net N$27: C22.2, GT2.P$1, R23.2
- net +5V: now also D7.A, U$2.5; no longer IC6.5
- net AUXGATE: now also RSOUT.1; no longer GX.1
- net GND: now also C22.1, CKI.P$3, CKO.P$3, CVA.P$3, CVB.P$3, CVC.P$3, CVD.P$3, D8.C, GD3.1, GD4.1, GT1.P$3, GT2.P$3, GT3.P$3, GT4.P$3, MIDIOUT.S, R34.1, RSI.P$3, RSO.P$3, U$2.2; no longer CKIN.2, CKO.2, CVA.2, CVB.2, CVC.2, CVD.2, GND.1, GT1.2, GT2.2, GT3.2, GT4.2, IC6.3, MIDI_OUT.2
- net N$1: now also MIDIOUT.R; no longer MIDI_OUT.5
- net N$10: now also CVB.P$1; no longer CVB.4
- net N$11: now also CVA.P$1; no longer CVA.4
- net N$4: now also MIDIIN.T; no longer MIDI_IN.4
- net N$44: now also RSO.P$1; no longer CKO.4
- net N$45: now also CKO.P$1; no longer GT2.4
- net N$46: now also GT1.P$1; no longer GT1.4
- net N$47: now also GT4.P$1; no longer GT4.4
- net N$48: now also GT3.P$1; no longer GT3.4
- net N$53: now also U$2.1; no longer IC6.2
- net N$54: now also CKI.P$1; no longer CKIN.4
- net N$6: now also MIDIOUT.T; no longer MIDI_OUT.4
- net N$7: now also MIDIIN.R; no longer MIDI_IN.5
- net N$8: now also CVC.P$1; no longer CVC.4
- net N$9: now also CVD.P$1; no longer CVD.4
Routing:
- net N$25: track 0.00 -> 121.2 mm, vias 0 -> 2
- net N$23: track 0.00 -> 115.5 mm, vias 0 -> 2
- net N$27: track 0.00 -> 93.5 mm, vias 0 -> 2
- net N$44: track 67.9 -> 14.2 mm, vias 2 -> 0
- net MIDI_OUT: track 94.8 -> 142.1 mm, vias 1 -> 2
- net N$24: track 0.00 -> 44.8 mm, vias 0 -> 1
- net N$48: track 12.7 -> 55.9 mm, vias 0 -> 1
- net CLKIN: track 42.0 -> 0.00 mm, vias 2 -> 0
- net N$8: track 26.4 -> 66.3 mm, vias 1 -> 2
- net N$47: track 35.9 -> 73.8 mm, vias 0 -> 2
- net +10V: track 72.0 -> 36.9 mm, vias 3 -> 2
- net N$46: track 56.7 -> 89.3 mm, vias 2 -> 0
- net N$9: track 32.3 -> 64.8 mm, vias 1 -> 2
- net N$56: track 2.93 -> 33.0 mm, vias 0 -> 1
- net N$45: track 64.8 -> 35.0 mm, vias 2 -> 0
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Other:
- board size 155.7 x 39.1 mm -> 155.7 x 37.8 mm
- board text added: "noodlebox i/o board rev 3"
- board text removed: "hotchk155"
- board text removed: "matrix sequencer i/o board rev 2"

Commit message: V3 candidate
Parts:
- removed U$2: SN74LVC2G14, jason_eagle6:DBV_R-PDSO-G6
- added IC6: 4504D, 45xx:SO16
- C1: value 10u -> 100n; device rcl:SMC_A -> rcl:C0805
- C13: value (none) -> 20p; device rcl:E2,5-7 -> rcl:C0805
- C14, C16: device rcl:E2,5-7 -> rcl:C0805
- C15: value 470p -> (none)
- C17: value 100n -> (none)
- C19, C20, C22: value 100n -> (none); device rcl:C0805 -> rcl:E2,5-7
- C21: value 100n -> 470p
- C4: value (none) -> 10u; device rcl:C0805 -> rcl:SMC_A
- C5, C7, C9: value (none) -> 100n
- C6: value 20p -> 100n
- D2: value MBR0520LT -> 0805DIODE; device diode:SOD123 -> jasons_stuff:0805DIODE
- D5: value CGRM4001-G -> 0805DIODE; device diode:SOD-123_MINI-SMA -> jasons_stuff:0805DIODE
- D7: value 0805DIODE -> CGRM4001-G; device jasons_stuff:0805DIODE -> diode:SOD-123_MINI-SMA
- D8: value 0805DIODE -> MBR0520LT; device jasons_stuff:0805DIODE -> diode:SOD123
- IC2: value LM27675M5_CHARGEPUMP -> SN74LVC2G14; device jason_eagle6:SOT23-6 -> jason_eagle6:DBV_R-PDSO-G6
- IC3: value LM324D -> LM27675M5_CHARGEPUMP; device linear:SO14 -> jason_eagle6:SOT23-6
- IC4: value MCP4728_QUAD_DAC -> LM324D; device jason_eagle6:MSOP10 -> linear:SO14
- IC5: value 4504D -> MCP4728_QUAD_DAC; device 45xx:SO16 -> jason_eagle6:MSOP10
- IC7: value FDS8958B -> SP34063A_BOOST_REG
- IC8: value SP34063A_BOOST_REG -> FDS8958B
- MIDIIN, MIDIOUT: value VERTICAL_3_5MM_SOCKETTHONK -> VERTICAL_3_5MM_SOCKETASSS; device jason_eagle6:PJ301CM -> jason_eagle6:OFFSET-PINS
- R14, R15, R16, R7, R9: value 10k/0.1% -> 1k
- R18, R20, R21, R22, R23: value 1k -> 10k/0.1%
- R2: value 1k8 -> 220
- R25, R26: value 10k -> 10k/0.1%
- R32, R34: value 470k -> 10k
- R5: value 220 -> 1k8
- R6, R8: value 10k/0.1% -> 470k
- moved D8 118.2 mm to (150.9, 25.6), turned to 0 degrees
- moved R32 110.4 mm to (134.2, 36.4), turned to 180 degrees
- moved R34 110.4 mm to (134.2, 31.4), turned to 0 degrees
- moved R33 108.6 mm to (134.2, 33.9), turned to 180 degrees
- moved D6 105.9 mm to (45.7, 12.7)
- moved C16 87.7 mm to (66.3, 33.5), turned to 90 degrees
- moved R25 84.9 mm to (49.5, 25.9), turned to 270 degrees
- moved R27 84.5 mm to (50.5, 22.4)
- moved R26 82.8 mm to (52.1, 25.9), turned to 270 degrees
- moved C22 80.3 mm to (151.1, 11.5)
- moved D7 58.9 mm to (90.6, 6.73)
- moved C15 58.0 mm to (54.6, 25.9), turned to 270 degrees
- moved D5 56.3 mm to (34.3, 6.35)
- moved R6 50.3 mm to (26.7, 11.4), turned to 270 degrees
- moved R9 46.9 mm to (29.2, 6.35), turned to 90 degrees
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- renumbered RSI to AUXI, RSO to AUXO, U$1 to DC
Connections:
- net +10V: now also C2.+, C9.2, D6.C, IC3.5, IC6.16; no longer C1.+, C10.2, D2.C, IC2.5, IC5.16
- net +5V: now also C1.1, C18.1, C19.+, C4.+, D4.A, D6.A, IC2.5, IC3.1, IC6.1, IC6.13, R1.2, R4.2; no longer C11.1, C12.1, C13.+, C3.+, D2.A, D7.A, IC2.1, IC4.1, IC5.13, R2.2, R3.2, U$2.5
- net +9V: now also C14.1, C22.+, IC4.4, IC8.5; no longer C16.+, C9.1, IC3.4, IC7.5
- net AUXGATE: now also IC6.9; no longer IC5.9
- net CLKOUT: now also IC6.3; no longer IC5.3
- net GATE1: now also IC6.14; no longer IC5.14
- net GATE2: now also IC6.5; no longer IC5.5
- net GATE3: now also IC6.7; no longer IC5.7
- net GATE4: now also IC6.11; no longer IC5.11
- net GND: now also C1.2, C11.1, C12.1, C14.2, C18.2, C19.-, C2.-, C20.-, C21.2, C22.-, C4.-, C5.1, C6.1, C7.1, C9.1, D2.C, D5.C, D7.A, IC3.2, IC3.4, IC4.11, IC5.10, IC5.4, IC6.8, IC7.4, IC8.1, MIDIOUT.P$1, R18.1, R20.1, R22.1, R5.2, R6.1; no longer C1.-, C11.2, C12.2, C13.-, C14.-, C15.2, C16.-, C17.1, C18.1, C19.1, C20.1, C21.1, C22.1, C3.-, C9.2, D4.C, D5.A, D8.C, IC2.4, IC3.11, IC4.10, IC4.4, IC5.8, IC7.1, IC8.4, MIDIOUT.S, R15.1, R16.1, R34.1, R4.2, R7.1, U$2.2
- net MIDI_IN: now also R4.1; no longer R2.1
- net MIDI_OUT: now also R2.2; no longer R5.2
- net N$1: now also MIDIOUT.P$2, R1.1; no longer MIDIOUT.R, R3.1
- net N$10: now also R19.2, R21.2; no longer R10.2, R6.2
- net N$11: now also R23.2, R24.2; no longer R11.2, R9.2
- net N$12: now also C13.2, IC4.1, R16.1; no longer C6.2, IC3.1, R12.1
- net N$13: now also C15.2, IC4.7, R27.1; no longer C7.2, IC3.7, R13.1
- net N$14: now also C17.2, IC4.8, R24.1; no longer C5.2, IC3.8, R11.1
- net N$15: now also C16.2, IC4.14, R19.1; no longer C4.2, IC3.14, R10.1
- net N$17: now also C16.1, IC4.13, R20.2, R21.1; no longer C4.1, IC3.13, R6.1, R7.2
- net N$18: now also C17.1, IC4.9, R22.2, R23.1; no longer C5.1, IC3.9, R8.2, R9.1
- net N$19: now also IC6.10, R15.1; no longer IC5.10, R23.1
- net N$2: now also R3.2; no longer R1.2
- net N$20: now also C15.1, IC4.6, R25.1, R26.2; no longer C7.1, IC3.6, R16.2, R17.1
- net N$22: now also C13.1, IC4.2, R17.1, R18.2; no longer C6.1, IC3.2, R14.1, R15.2
- net N$23: now also IC2.6; no longer U$2.6
- net N$24: now also R8.2, R9.2; no longer R33.2, R34.2
- net N$25: now also IC2.4; no longer U$2.4
- net N$26: now also D4.C, D5.A, IC2.3, R9.1; no longer D7.C, D8.A, R33.1, U$2.3
- net N$27: now also C12.2, R15.2; no longer C22.2, R23.2
- net N$29: now also IC4.5, IC5.6; no longer IC3.5, IC4.6
- net N$3: now also IC4.3, IC5.7; no longer IC3.3, IC4.7
- net N$30: now also IC4.10, IC5.9; no longer IC3.10, IC4.9
- net N$31: now also IC4.12, IC5.8; no longer IC3.12, IC4.8
- net N$32: now also IC7.1, IC7.7, IC7.8; no longer IC8.1, IC8.7, IC8.8
- net N$33: now also IC7.5; no longer IC8.5
- net N$34: now also C21.1, IC7.3; no longer C15.1, IC8.3
- net N$35: now also D7.C, IC7.2; no longer D5.C, IC8.2
- net N$36: now also D8.A; no longer D6.A
- net N$37: now also IC6.2, R10.1; no longer IC5.2, R18.1
- net N$38: now also C3.+, IC3.6; no longer C2.+, IC2.6
- net N$39: now also C3.-, IC3.3; no longer C2.-, IC2.3
- net N$4: now also MIDIIN.P$3; no longer MIDIIN.T
- net N$40: now also IC6.4, R11.1; no longer IC5.4, R19.1
- net N$41: now also IC6.6, R12.1; no longer IC5.6, R20.1
- net N$43: now also IC6.12, R14.1; no longer IC5.12, R22.1
- net N$44: now also C5.2, R10.2; no longer C17.2, R18.2
- net N$45: now also C6.2, R11.2; no longer C18.2, R19.2
- net N$46: now also C7.2, R12.2; no longer C19.2, R20.2
- net N$47: now also C11.2, R14.2; no longer C20.2, R22.2
- net N$48: now also C10.2, R13.2; no longer C21.2, R21.2
- net N$49: now also IC6.15, R13.1; no longer IC5.15, R21.1
- net N$5: now also R5.1; no longer R4.1
- net N$51: now also C20.+; no longer C14.+
- net N$53: now also D2.A, IC2.1, R7.1; no longer D4.A, R24.1, U$2.1
- net N$54: now also R6.2, R7.2; no longer R24.2, R32.2
- net N$6: now also MIDIOUT.P$3, R2.1; no longer MIDIOUT.T, R5.1
- net N$61: now also IC8.4, IC8.7, IC8.8, R34.2; no longer IC7.4, IC7.7, IC7.8, R25.2
- net N$62: now also IC8.2, R32.2, R33.2; no longer IC7.2, R26.2, R27.2
- net N$7: now also MIDIIN.P$2, R3.1; no longer MIDIIN.R, R1.1
- net N$8: now also R16.2, R17.2; no longer R12.2, R14.2
- net N$9: now also R25.2, R27.2; no longer R13.2, R17.2
- net PWR_CTRL: now also R33.1; no longer R27.1
- net SCL: now also IC5.2; no longer IC4.2
- net SDA: now also IC5.3; no longer IC4.3
- net VIN: now also D8.C, IC8.3, R34.1; no longer D6.C, IC7.3, R25.1
Routing:
- net N$1: track 27.6 -> 12.0 mm
- net N$6: track 22.6 -> 11.6 mm
- net N$7: track 13.3 -> 23.5 mm, vias 0 -> 1
- net N$4: track 26.1 -> 30.4 mm
- net MIDI_OUT: track 142.1 -> 140.2 mm
- net +5V: track 223.2 -> 224.7 mm, vias 7 -> 6
Other:
- board text added: "NOODLEBOX I/O BOARD V3"
- board text removed: "noodlebox i/o board rev 3"

Commit message: values
Parts:
- R6, R8: value 470k -> 100k
Changed lines of the file:
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@@
 <attribute name="VALUE" x="142.24" y="9.525" size="1.27" layer="27"/>
 </element>
-<element name="R6" library="rcl" package="R0805" value="470k" x="26.67" y="11.43" smashed="yes" rot="R270">
+<element name="R6" library="rcl" package="R0805" value="100k" x="26.67" y="11.43" smashed="yes" rot="R270">
 <attribute name="NAME" x="25.908" y="13.843" size="1.016" layer="25" font="vector" ratio="20"/>
 </element>
@@
 <attribute name="NAME" x="30.353" y="3.937" size="1.016" layer="25" font="vector" ratio="20" rot="R180"/>
 </element>
-<element name="R8" library="rcl" package="R0805" value="470k" x="26.67" y="6.35" smashed="yes" rot="R90">
+<element name="R8" library="rcl" package="R0805" value="100k" x="26.67" y="6.35" smashed="yes" rot="R90">
 <attribute name="NAME" x="27.686" y="3.937" size="1.016" layer="25" font="vector" ratio="20" rot="R180"/>
 </element>
