File: matrix_io_board.sch (EAGLE design)
At the start: 101 parts, among them IC1 6N138, IC2 LM27675M5_CHARGEPUMP, IC3 LM324D, IC4 MCP4728_QUAD_DAC, IC5 4504D, IC6 74AHC1G14DBV, IC7 FDS8958B, IC8 SP34063A_BOOST_REG

Commit message: rename
Parts:
- GD2: value GD -> (none)
- renumbered 5V1 to 5V., GND26 to GD1, GND38 to GD2
Changed lines of the file:
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@@
 <part name="P+15" library="supply1" deviceset="+5V" device=""/>
 <part name="GND30" library="supply1" deviceset="GND" device=""/>
-<part name="GND38" library="pinhead" deviceset="PINHD-1X1" device="" value="GD"/>
+<part name="GD2" library="pinhead" deviceset="PINHD-1X1" device=""/>
 <part name="GND40" library="supply1" deviceset="GND" device=""/>
 <part name="L1" library="SparkFun" deviceset="INDUCTOR" device="1210"/>
@@
 <part name="PWRCTL" library="pinhead" deviceset="PINHD-1X1" device=""/>
 <part name="AUX" library="microbuilder" deviceset="TESTPOINT" device="ROUND2MM"/>
-<part name="GND26" library="pinhead" deviceset="PINHD-1X1" device="" value="GD"/>
-<part name="5V1" library="pinhead" deviceset="PINHD-1X1" device=""/>
+<part name="GD1" library="pinhead" deviceset="PINHD-1X1" device="" value="GD"/>
+<part name="5V." library="pinhead" deviceset="PINHD-1X1" device=""/>
 <part name="OFFSW" library="pinhead" deviceset="PINHD-1X1" device=""/>
 </parts>
@@
 <instance part="P+15" gate="1" x="421.64" y="347.98"/>
 <instance part="GND30" gate="1" x="421.64" y="307.34"/>
-<instance part="GND38" gate="G$1" x="414.02" y="320.04" rot="R180"/>
+<instance part="GD2" gate="G$1" x="414.02" y="320.04" rot="R180"/>
 <instance part="GND40" gate="1" x="109.22" y="165.1"/>
 <instance part="L1" gate="G$1" x="271.78" y="317.5" rot="R90"/>
@@
 <instance part="PWRCTL" gate="G$1" x="99.06" y="330.2" rot="R180"/>
 <instance part="AUX" gate="G$1" x="388.62" y="228.6" rot="R180"/>
-<instance part="GND26" gate="G$1" x="414.02" y="312.42" rot="R180"/>
-<instance part="5V1" gate="G$1" x="414.02" y="342.9" rot="R180"/>
+<instance part="GD1" gate="G$1" x="414.02" y="312.42" rot="R180"/>
+<instance part="5V." gate="G$1" x="414.02" y="342.9" rot="R180"/>
 <instance part="OFFSW" gate="G$1" x="269.24" y="170.18"/>
 </instances>
@@
 <wire x1="416.56" y1="327.66" x2="421.64" y2="327.66" width="0.1524" layer="91"/>
 <wire x1="421.64" y1="327.66" x2="421.64" y2="320.04" width="0.1524" layer="91"/>
-<pinref part="GND38" gate="G$1" pin="1"/>
+<pinref part="GD2" gate="G$1" pin="1"/>
 <wire x1="421.64" y1="320.04" x2="421.64" y2="312.42" width="0.1524" layer="91"/>
 <wire x1="421.64" y1="312.42" x2="421.64" y2="309.88" width="0.1524" layer="91"/>
 <wire x1="416.56" y1="320.04" x2="421.64" y2="320.04" width="0.1524" layer="91"/>
 <junction x="421.64" y="320.04"/>
-<pinref part="GND26" gate="G$1" pin="1"/>
+<pinref part="GD1" gate="G$1" pin="1"/>
 <wire x1="416.56" y1="312.42" x2="421.64" y2="312.42" width="0.1524" layer="91"/>
 <junction x="421.64" y="312.42"/>
@@
 <wire x1="416.56" y1="335.28" x2="421.64" y2="335.28" width="0.1524" layer="91"/>
 <wire x1="421.64" y1="335.28" x2="421.64" y2="342.9" width="0.1524" layer="91"/>
-<pinref part="5V1" gate="G$1" pin="1"/>
+<pinref part="5V." gate="G$1" pin="1"/>
 <wire x1="421.64" y1="342.9" x2="421.64" y2="345.44" width="0.1524" layer="91"/>
 <wire x1="416.56" y1="342.9" x2="421.64" y2="342.9" width="0.1524" layer="91"/>

Commit message: changes for rev2
Parts:
- removed AUX: (no value), microbuilder:TESTPOINTROUND2MM
- removed GATE: (no value), pinhead:PINHD-2X3
- removed R23: (no value), rcl:R-EU_R0805
- added C17, C18, C19, C20, C21: 100n, rcl:C-EUC0805
- added R32: 470k, rcl:R-EU_R0805
- C1, C2, C3: value (none) -> 10u
- C10, C11, C12, C8: value (none) -> 100n
- C15: value (none) -> 470p
- C6: value (none) -> 20p
- R1, R3, R5: value (none) -> 220
- R10, R11, R12, R13, R18, R19, R20, R21, R22, R24, R27, R28, R30: value (none) -> 1k
- R14, R15, R16, R17, R6, R7, R8, R9: value (none) -> 10k/0.1%
- R2, R4: value (none) -> 1k8
- R25, R26: value (none) -> 10k
- R29: value (none) -> 0r33
- R31: value (none) -> 3k
Connections:
- removed net N$42: IC5A.DO, R23.1
- removed net N$50: AUX.P$1, R23.2
- removed net N$71: BATT-.1, U$1.NC
- removed net VGATE: C10.2, GATE.1, GATE.3, GATE.5, IC5P.VDD
- new net N$16: BATT+.1, U$1.NC
- net +10V: now also C10.2, IC5P.VDD; no longer GATE.4
- net +5V: no longer GATE.2
- net +9V: no longer GATE.6
- net GND: now also BATT-.1, C17.1, C18.1, C19.1, C20.1, C21.1, R32.1, U$1.PIN; no longer U$1.BARREL
- net N$36: now also U$1.BARREL; no longer BATT+.1, U$1.PIN
- net N$44: now also C17.2
- net N$45: now also C18.2
- net N$46: now also C19.2
- net N$47: now also C20.2
- net N$48: now also C21.2
- net N$54: now also R32.2
Other:
- note added: "Rev 2 -19 May 19 - Sixty Four Pixels Ltd"
- note removed: "Rev 1 - April 2018 - Sixty Four Pixels Ltd"
- moved on the sheet: CKIN, CKO, GT1, GT2, GT3, GT4

Commit message: work in progress
Parts:
- removed CKIN: VERTICAL_3_5MM_SOCKET, jason_eagle6:VERTICAL_3_5MM_SOCKET
- removed GND: (no value), pinhead:PINHD-1X1
- removed IC6: 74AHC1G14DBV, 74xx-little-de:74AHC1G14DBV
- removed MIDI_IN, MIDI_OUT: DIN5PIN, jason_eagle6:DIN5PIN
- added C22: 100n, rcl:C-EUC0805
- added CKI, RSI, RSO: WQP-PJ301M-12_JACK, thonkiconn:WQP-PJ301M-12_JACK
- added D7, D8: 0805DIODE, jasons_stuff:0805DIODE
- added GD3, GD4, RSIN: (no value), pinhead:PINHD-1X1
- added MIDIIN, MIDIOUT: VERTICAL_3_5MM_SOCKETTHONK, jason_eagle6:VERTICAL_3_5MM_SOCKETTHONK
- added R23, R33: 1k, rcl:R-EU_R0805
- added R34: 470k, rcl:R-EU_R0805
- added U$2: SN74LVC2G14, jason_eagle6:SN74LVC2G14
- CKO, CVA, CVB, CVC, CVD, GT1, GT2, GT3, GT4: value VERTICAL_3_5MM_SOCKET -> WQP-PJ301M-12_JACK; device jason_eagle6:VERTICAL_3_5MM_SOCKET -> thonkiconn:WQP-PJ301M-12_JACK
- GD1: value GD -> (none)
- L2: device inductors:DR1030 -> jason_eagle6:NB_IND
- renumbered GX to RSOUT
Connections:
- removed net CLKIN: CLKIN.1, IC6A.O
- new net N$19: IC5A.DO, R23.1
- new net N$23: CLKIN.1, U$2.1Y
- new net N$24: R33.2, R34.2, RSI.2
- new net N$25: RSIN.1, U$2.2Y
- new net N$26: D7.P$1, D8.P$2, R33.1, U$2.2A
- new net N$27: C22.2, GT2.2, R23.2
- net +5V: now also D7.P$2, U$2.VCC; no longer IC6P.VCC
- net GND: now also C22.1, CKI.1, CKO.1, CVA.1, CVB.1, CVC.1, CVD.1, D8.P$1, GD3.1, GD4.1, GT1.1, GT2.1, GT3.1, GT4.1, MIDIOUT.2, R34.1, RSI.1, RSO.1, U$2.GND; no longer CKIN.2, CKO.2, CVA.2, CVB.2, CVC.2, CVD.2, GND.1, GT1.2, GT2.2, GT3.2, GT4.2, IC6P.GND, MIDI_OUT.2
- net N$1: now also MIDIOUT.3; no longer MIDI_OUT.5
- net N$10: now also CVB.2; no longer CVB.4
- net N$11: now also CVA.2; no longer CVA.4
- net N$4: now also MIDIIN.4; no longer MIDI_IN.4
- net N$44: now also RSO.2; no longer CKO.4
- net N$45: now also CKO.2; no longer GT2.4
- net N$46: now also GT1.2; no longer GT1.4
- net N$47: now also GT4.2; no longer GT4.4
- net N$48: now also GT3.2; no longer GT3.4
- net N$53: now also U$2.1A; no longer IC6A.I
- net N$54: now also CKI.2; no longer CKIN.4
- net N$6: now also MIDIOUT.4; no longer MIDI_OUT.4
- net N$7: now also MIDIIN.3; no longer MIDI_IN.5
- net N$8: now also CVC.2; no longer CVC.4
- net N$9: now also CVD.2; no longer CVD.4
Other:
- moved on the sheet: C12, CLKIN, GD1, GD2, R24, R32

Commit message: V3 candidate
Parts:
- removed U$2: SN74LVC2G14, jason_eagle6:SN74LVC2G14
- added IC6: 4504D, 45xx:4504D
- C1: value 10u -> 100n; device rcl:CPOL-EUSMCA -> rcl:C-EUC0805
- C13: value (none) -> 20p; device rcl:CPOL-EUE2.5-7 -> rcl:C-EUC0805
- C14, C16: device rcl:CPOL-EUE2.5-7 -> rcl:C-EUC0805
- C15: value 470p -> (none)
- C17: value 100n -> (none)
- C19, C20, C22: value 100n -> (none); device rcl:C-EUC0805 -> rcl:CPOL-EUE2.5-7
- C21: value 100n -> 470p
- C4: value (none) -> 10u; device rcl:C-EUC0805 -> rcl:CPOL-EUSMCA
- C5, C7, C9: value (none) -> 100n
- C6: value 20p -> 100n
- D2: value MBR0520LT -> 0805DIODE; device diode:MBR0520LT -> jasons_stuff:0805DIODE
- D5: value CGRM4001-G -> 0805DIODE; device diode:CGRM4001-G -> jasons_stuff:0805DIODE
- D7: value 0805DIODE -> CGRM4001-G; device jasons_stuff:0805DIODE -> diode:CGRM4001-G
- D8: value 0805DIODE -> MBR0520LT; device jasons_stuff:0805DIODE -> diode:MBR0520LT
- IC2: value LM27675M5_CHARGEPUMP -> SN74LVC2G14; device jason_eagle6:LM27675M5_CHARGEPUMP -> jason_eagle6:SN74LVC2G14
- IC3: value LM324D -> LM27675M5_CHARGEPUMP; device linear:LM324D -> jason_eagle6:LM27675M5_CHARGEPUMP
- IC4: value MCP4728_QUAD_DAC -> LM324D; device jason_eagle6:MCP4728_QUAD_DAC -> linear:LM324D
- IC5: value 4504D -> MCP4728_QUAD_DAC; device 45xx:4504D -> jason_eagle6:MCP4728_QUAD_DAC
- IC7: value FDS8958B -> SP34063A_BOOST_REG; device jason_eagle6:FDS8958B -> jason_eagle6:SP34063A_BOOST_REG
- IC8: value SP34063A_BOOST_REG -> FDS8958B; device jason_eagle6:SP34063A_BOOST_REG -> jason_eagle6:FDS8958B
- MIDIIN, MIDIOUT: value VERTICAL_3_5MM_SOCKETTHONK -> VERTICAL_3_5MM_SOCKETASSS; device jason_eagle6:VERTICAL_3_5MM_SOCKETTHONK -> jason_eagle6:VERTICAL_3_5MM_SOCKETASSS
- R14, R15, R16, R7, R9: value 10k/0.1% -> 1k
- R18, R20, R21, R22, R23: value 1k -> 10k/0.1%
- R2: value 1k8 -> 220
- R25, R26: value 10k -> 10k/0.1%
- R32, R34: value 470k -> 10k
- R5: value 220 -> 1k8
- R6, R8: value 10k/0.1% -> 470k
- renumbered RSI to AUXI, RSO to AUXO, U$1 to DC
Connections:
- net +10V: now also C2.+, C9.2, D6.C, IC3.OUT, IC6P.VDD; no longer C1.+, C10.2, D2.C, IC2.OUT, IC5P.VDD
- net +5V: now also C1.1, C18.1, C19.+, C4.+, D4.P$2, D6.A, IC2.VCC, IC3.V+, IC5.VDD, IC6A.MODE, IC6P.VCC, R1.2, R4.2; no longer C11.1, C12.1, C13.+, C3.+, D2.A, D7.P$2, IC2.V+, IC4.VDD, IC5A.MODE, IC5P.VCC, R2.2, R3.2, U$2.VCC
- net +9V: now also C14.1, C22.+, IC4P.V+, IC7.VCC, IC8.D2, IC8.D2@; no longer C16.+, C9.1, IC3P.V+, IC7.D2, IC7.D2@, IC8.VCC
- net AUXGATE: now also IC6A.DI; no longer IC5A.DI
- net CLKOUT: now also IC6A.AI; no longer IC5A.AI
- net GATE1: now also IC6A.FI; no longer IC5A.FI
- net GATE2: now also IC6A.BI; no longer IC5A.BI
- net GATE3: now also IC6A.CI; no longer IC5A.CI
- net GATE4: now also IC6A.EI; no longer IC5A.EI
- net GND: now also C1.2, C11.1, C12.1, C14.2, C18.2, C19.-, C2.-, C20.-, C21.2, C22.-, C4.-, C5.1, C6.1, C7.1, C9.1, D2.P$1, D5.P$1, D7.A, IC3.GND, IC3.SD, IC4P.V-, IC5.LDAC#, IC5.VSS, IC6P.GND, IC7.GND, IC8.S1, R18.1, R20.1, R22.1, R5.2, R6.1; no longer C1.-, C11.2, C12.2, C13.-, C14.-, C15.2, C16.-, C17.1, C18.1, C19.1, C20.1, C21.1, C22.1, C3.-, C9.2, D4.P$1, D5.A, D8.P$1, IC2.SD, IC3P.V-, IC4.LDAC#, IC4.VSS, IC5P.GND, IC7.S1, IC8.GND, R15.1, R16.1, R34.1, R4.2, R7.1, U$2.GND
- net MIDI_IN: now also R4.1; no longer R2.1
- net MIDI_OUT: now also R2.2; no longer R5.2
- net N$1: now also R1.1; no longer R3.1
- net N$10: now also R19.2, R21.2; no longer R10.2, R6.2
- net N$11: now also R23.2, R24.2; no longer R11.2, R9.2
- net N$12: now also C13.2, IC4A.OUT, R16.1; no longer C6.2, IC3A.OUT, R12.1
- net N$13: now also C15.2, IC4B.OUT, R27.1; no longer C7.2, IC3B.OUT, R13.1
- net N$14: now also C17.2, IC4C.OUT, R24.1; no longer C5.2, IC3C.OUT, R11.1
- net N$15: now also C16.2, IC4D.OUT, R19.1; no longer C4.2, IC3D.OUT, R10.1
- net N$17: now also C16.1, IC4D.-IN, R20.2, R21.1; no longer C4.1, IC3D.-IN, R6.1, R7.2
- net N$18: now also C17.1, IC4C.-IN, R22.2, R23.1; no longer C5.1, IC3C.-IN, R8.2, R9.1
- net N$19: now also IC6A.DO, R15.1; no longer IC5A.DO, R23.1
- net N$2: now also R3.2; no longer R1.2
- net N$20: now also C15.1, IC4B.-IN, R25.1, R26.2; no longer C7.1, IC3B.-IN, R16.2, R17.1
- net N$22: now also C13.1, IC4A.-IN, R17.1, R18.2; no longer C6.1, IC3A.-IN, R14.1, R15.2
- net N$23: now also IC2.1Y; no longer U$2.1Y
- net N$24: now also R8.2, R9.2; no longer R33.2, R34.2
- net N$25: now also IC2.2Y; no longer U$2.2Y
- net N$26: now also D4.P$1, D5.P$2, IC2.2A, R9.1; no longer D7.P$1, D8.P$2, R33.1, U$2.2A
- net N$27: now also C12.2, R15.2; no longer C22.2, R23.2
- net N$29: now also IC4B.+IN, IC5.VOUTA; no longer IC3B.+IN, IC4.VOUTA
- net N$3: now also IC4A.+IN, IC5.VOUTB; no longer IC3A.+IN, IC4.VOUTB
- net N$30: now also IC4C.+IN, IC5.VOUTD; no longer IC3C.+IN, IC4.VOUTD
- net N$31: now also IC4D.+IN, IC5.VOUTC; no longer IC3D.+IN, IC4.VOUTC
- net N$32: now also IC7.DR_C, IC7.SENS, IC7.SW_C; no longer IC8.DR_C, IC8.SENS, IC8.SW_C
- net N$33: now also IC7.COMP; no longer IC8.COMP
- net N$34: now also C21.1, IC7.TC; no longer C15.1, IC8.TC
- net N$35: now also D7.C, IC7.SW_E; no longer D5.C, IC8.SW_E
- net N$36: now also D8.A; no longer D6.A
- net N$37: now also IC6A.AO, R10.1; no longer IC5A.AO, R18.1
- net N$38: now also C3.+, IC3.CAP+; no longer C2.+, IC2.CAP+
- net N$39: now also C3.-, IC3.CAP-; no longer C2.-, IC2.CAP-
- net N$40: now also IC6A.BO, R11.1; no longer IC5A.BO, R19.1
- net N$41: now also IC6A.CO, R12.1; no longer IC5A.CO, R20.1
- net N$43: now also IC6A.EO, R14.1; no longer IC5A.EO, R22.1
- net N$44: now also C5.2, R10.2; no longer C17.2, R18.2
- net N$45: now also C6.2, R11.2; no longer C18.2, R19.2
- net N$46: now also C7.2, R12.2; no longer C19.2, R20.2
- net N$47: now also C11.2, R14.2; no longer C20.2, R22.2
- net N$48: now also C10.2, R13.2; no longer C21.2, R21.2
- net N$49: now also IC6A.FO, R13.1; no longer IC5A.FO, R21.1
- net N$5: now also R5.1; no longer R4.1
- net N$51: now also C20.+; no longer C14.+
- net N$53: now also D2.P$2, IC2.1A, R7.1; no longer D4.P$2, R24.1, U$2.1A
- net N$54: now also R6.2, R7.2; no longer R24.2, R32.2
- net N$6: now also R2.1; no longer R5.1
- net N$61: now also IC8.D1, IC8.D1@, IC8.G2, R34.2; no longer IC7.D1, IC7.D1@, IC7.G2, R25.2
- net N$62: now also IC8.G1, R32.2, R33.2; no longer IC7.G1, R26.2, R27.2
- net N$7: now also R3.1; no longer R1.1
- net N$8: now also R16.2, R17.2; no longer R12.2, R14.2
- net N$9: now also R25.2, R27.2; no longer R13.2, R17.2
- net PWR_CTRL: now also R33.1; no longer R27.1
- net SCL: now also IC5.SCL; no longer IC4.SCL
- net SDA: now also IC5.SDA; no longer IC4.SDA
- net VIN: now also D8.C, IC8.S2, R34.1; no longer D6.C, IC7.S2, R25.1
Other:
- note added: "NOODLEBOX I/O AND POWER BOARD"
- note added: "Rev 3 -26 Nov19 - Sixty Four Pixels Ltd"
- note removed: "MATRIX SEQUENCER I/O AND POWER BOARD"
- note removed: "Rev 2 -19 May 19 - Sixty Four Pixels Ltd"
- moved on the sheet: C10, C11, C12, C15, C17, C18, C2, C21, C3, C5, C6, C7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

Commit message: values
Parts:
- R6, R8: value 470k -> 100k
Changed lines of the file:
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@@
 <part name="5V." library="pinhead" deviceset="PINHD-1X1" device=""/>
 <part name="OFFSW" library="pinhead" deviceset="PINHD-1X1" device=""/>
-<part name="R6" library="rcl" deviceset="R-EU_" device="R0805" value="470k"/>
+<part name="R6" library="rcl" deviceset="R-EU_" device="R0805" value="100k"/>
 <part name="GND26" library="supply1" deviceset="GND" device=""/>
 <part name="C5" library="rcl" deviceset="C-EU" device="C0805" value="100n"/>
@@
 <part name="R9" library="rcl" deviceset="R-EU_" device="R0805" value="1k"/>
 <part name="GND20" library="supply1" deviceset="GND" device=""/>
-<part name="R8" library="rcl" deviceset="R-EU_" device="R0805" value="470k"/>
+<part name="R8" library="rcl" deviceset="R-EU_" device="R0805" value="100k"/>
 <part name="D4" library="jasons_stuff" deviceset="0805DIODE" device=""/>
 <part name="D5" library="jasons_stuff" deviceset="0805DIODE" device=""/>
