File: matrix_io_board.sch (EAGLE design)
At the start: 114 parts, among them IC1 6N138, IC2 SN74LVC2G14, IC3 LM27675M5_CHARGEPUMP, IC4 LM324D, IC5 MCP4728_QUAD_DAC, IC6 4504D, IC7 SP34063A_BOOST_REG, IC8 FDS8958B

Commit message: 3v3 updates
Parts:
- removed C19, C20, C22: (no value), rcl:CPOL-EUD
- removed C2, C3, C4: 10u, rcl:CPOL-EUSMCA
- removed C21: 470p, rcl:C-EUC0805
- removed D6, D7: MBR0520LT, diode:MBR0520LT
- removed GD1, GD2: (no value), pinhead:PINHD-1X1
- removed IC3: LM27675M5_CHARGEPUMP, jason_eagle6:LM27675M5_CHARGEPUMP
- removed IC7: SP34063A_BOOST_REG, jason_eagle6:SP34063A_BOOST_REG
- removed IC8: FDS8958B, jason_eagle6:FDS8958B
- removed L1: (no value), SparkFun:INDUCTOR1210
- removed L2: (no value), jason_eagle6:NB_IND
- removed R31: 3k, rcl:R-EU_R0805
- removed R32, R34: 10k, rcl:R-EU_R0805
- removed R33: 1k, rcl:R-EU_R0805
- added C23, C24: 1u, rcl:C-EUC0805
- added C25, C26, C27, C32: 100n, rcl:C-EUC0805
- added C28, C29, C30, C31: (no value), rcl:CPOL-EUD
- added D+, D-: (no value), pinhead:PINHD-1X1
- added D10, D11, D9: MBR0520LT, diode:MBR0520LT
- added IC10, IC9: REG1117, burr-brown:REG1117
- added IC12: AP3012, jason2:AP3012
- added J1: 1734753-1, jason2:1734753-1
- added Q1: FDN360P, transistor-power:FDN360P
- added R35, R36: 1k, rcl:R-EU_R0805
- added T1: (no value), transistor:MMBT3904LT1-NPN-SOT23-BEC
- added U$2: CDRH3D14, jason2:CDRH3D14
- R29: value 0r33 -> (none)
- R30: value 1k -> (none)
- renumbered 5V to 3V, 5V. to 3V.
Connections:
- removed net +5V: 3V..1, 3V.1, C1.1, C18.1, C19.+, C4.+, C8.1, D3.P$2, D4.P$2, D6.A, IC1.VCC, IC2.VCC, IC3.V+, IC5.VDD, IC6A.MODE, IC6P.VCC, L1.2, R1.2, R28.1, R4.2
- removed net +9V: C14.1, C22.+, IC4P.V+, IC7.VCC, IC8.D2, IC8.D2@, R29.1
- removed net N$39: C3.-, IC3.CAP-
- removed net N$51: C20.+, L1.1, L2.1, R31.1
- removed net N$61: IC8.D1, IC8.D1@, IC8.G2, ON.S1, R34.2
- removed net N$62: IC8.G1, R32.2, R33.2
- removed net PWR_CTRL: PWRCTL.1, R33.1
- removed net VIN: D8.C, IC8.S2, R34.1
- new net +3V3: 3V..1, 3V.1, C1.1, C18.1, C31.+, C32.2, C8.1, D3.P$2, D4.P$2, IC1.VCC, IC10.VOUT, IC2.VCC, IC5.VDD, IC6A.MODE, IC6P.VCC, R1.2, R28.1, R4.2
- new net N$21: C26.2, C29.+, D10.A, IC9.VOUT
- new net N$28: D9.A, IC12.SW, U$2.P$1
- new net N$42: PWRCTL.1, R30.2
- new net N$52: IC12.FB, R35.1, R36.2
- new net USB_DM: D-.1, J1.2
- new net USB_DP: D+.1, J1.3
- new net VUSB: D11.A, J1.1
- net +10V: now also C14.1, C23.2, D9.C, IC4P.V+, R35.2; no longer C2.+, D6.C, IC3.OUT
- net GND: now also C23.1, C24.1, C25.1, C26.1, C27.1, C28.-, C29.-, C30.-, C31.-, C32.1, IC10.GND, IC12.GND, IC9.GND, J1.5, ON.S, ON.S1, R36.1, T1.E; no longer C19.-, C2.-, C20.-, C21.2, C22.-, C4.-, D7.A, GD1.1, GD2.1, IC3.GND, IC3.SD, IC7.GND, IC8.S1, ON.P, R30.1, R32.1
- net N$32: now also D10.C, D11.C, Q1.S; no longer IC7.DR_C, IC7.SENS, IC7.SW_C
- net N$33: now also C24.2, C27.2, C30.+, IC10.VIN, IC12.SHDN#, IC12.VIN, Q1.D, U$2.P$2; no longer IC7.COMP, R30.2, R31.2
- net N$34: now also ON.P, ON.P1, Q1.G, R29.1, T1.C; no longer C21.1, IC7.TC
- net N$35: now also R30.1, T1.B; no longer D7.C, IC7.SW_E, L2.2
- net N$38: now also C25.2, C28.+, D8.C, IC9.VIN; no longer C3.+, IC3.CAP+
Other:
- note removed: "10V CHARGE PUMP"
- note removed: "POWER SUPPLY"
- note removed: "SOFT SWITCH"
- moved on the sheet: BT+, BT-, D8, OFF, OFFSW, ON, PWR, PWRCTL, R28, R29, R30

Commit message: Revert "3v3 updates"
This reverts commit 782c7fb22120100be74f5025aa682998f87b6e62.
Parts:
- removed C23, C24: 1u, rcl:C-EUC0805
- removed C25, C26, C27, C32: 100n, rcl:C-EUC0805
- removed C28, C29, C30, C31: (no value), rcl:CPOL-EUD
- removed D+, D-: (no value), pinhead:PINHD-1X1
- removed D10, D11, D9: MBR0520LT, diode:MBR0520LT
- removed IC10, IC9: REG1117, burr-brown:REG1117
- removed IC12: AP3012, jason2:AP3012
- removed J1: 1734753-1, jason2:1734753-1
- removed Q1: FDN360P, transistor-power:FDN360P
- removed R35, R36: 1k, rcl:R-EU_R0805
- removed T1: (no value), transistor:MMBT3904LT1-NPN-SOT23-BEC
- removed U$2: CDRH3D14, jason2:CDRH3D14
- added C19, C20, C22: (no value), rcl:CPOL-EUD
- added C2, C3, C4: 10u, rcl:CPOL-EUSMCA
- added C21: 470p, rcl:C-EUC0805
- added D6, D7: MBR0520LT, diode:MBR0520LT
- added GD1, GD2: (no value), pinhead:PINHD-1X1
- added IC3: LM27675M5_CHARGEPUMP, jason_eagle6:LM27675M5_CHARGEPUMP
- added IC7: SP34063A_BOOST_REG, jason_eagle6:SP34063A_BOOST_REG
- added IC8: FDS8958B, jason_eagle6:FDS8958B
- added L1: (no value), SparkFun:INDUCTOR1210
- added L2: (no value), jason_eagle6:NB_IND
- added R31: 3k, rcl:R-EU_R0805
- added R32, R34: 10k, rcl:R-EU_R0805
- added R33: 1k, rcl:R-EU_R0805
- R29: value (none) -> 0r33
- R30: value (none) -> 1k
- renumbered 3V to 5V, 3V. to 5V.
Connections:
- removed net +3V3: 5V..1, 5V.1, C1.1, C18.1, C31.+, C32.2, C8.1, D3.P$2, D4.P$2, IC1.VCC, IC10.VOUT, IC2.VCC, IC5.VDD, IC6A.MODE, IC6P.VCC, R1.2, R28.1, R4.2
- removed net N$21: C26.2, C29.+, D10.A, IC9.VOUT
- removed net N$28: D9.A, IC12.SW, U$2.P$1
- removed net N$42: PWRCTL.1, R30.2
- removed net N$52: IC12.FB, R35.1, R36.2
- removed net USB_DM: D-.1, J1.2
- removed net USB_DP: D+.1, J1.3
- removed net VUSB: D11.A, J1.1
- new net +5V: 5V..1, 5V.1, C1.1, C18.1, C19.+, C4.+, C8.1, D3.P$2, D4.P$2, D6.A, IC1.VCC, IC2.VCC, IC3.V+, IC5.VDD, IC6A.MODE, IC6P.VCC, L1.2, R1.2, R28.1, R4.2
- new net +9V: C14.1, C22.+, IC4P.V+, IC7.VCC, IC8.D2, IC8.D2@, R29.1
- new net N$39: C3.-, IC3.CAP-
- new net N$51: C20.+, L1.1, L2.1, R31.1
- new net N$61: IC8.D1, IC8.D1@, IC8.G2, ON.S1, R34.2
- new net N$62: IC8.G1, R32.2, R33.2
- new net PWR_CTRL: PWRCTL.1, R33.1
- new net VIN: D8.C, IC8.S2, R34.1
- net +10V: now also C2.+, D6.C, IC3.OUT; no longer C14.1, C23.2, D9.C, IC4P.V+, R35.2
- net GND: now also C19.-, C2.-, C20.-, C21.2, C22.-, C4.-, D7.A, GD1.1, GD2.1, IC3.GND, IC3.SD, IC7.GND, IC8.S1, ON.P, R30.1, R32.1; no longer C23.1, C24.1, C25.1, C26.1, C27.1, C28.-, C29.-, C30.-, C31.-, C32.1, IC10.GND, IC12.GND, IC9.GND, J1.5, ON.S, ON.S1, R36.1, T1.E
- net N$32: now also IC7.DR_C, IC7.SENS, IC7.SW_C; no longer D10.C, D11.C, Q1.S
- net N$33: now also IC7.COMP, R30.2, R31.2; no longer C24.2, C27.2, C30.+, IC10.VIN, IC12.SHDN#, IC12.VIN, Q1.D, U$2.P$2
- net N$34: now also C21.1, IC7.TC; no longer ON.P, ON.P1, Q1.G, R29.1, T1.C
- net N$35: now also D7.C, IC7.SW_E, L2.2; no longer R30.1, T1.B
- net N$38: now also C3.+, IC3.CAP+; no longer C25.2, C28.+, D8.C, IC9.VIN
Other:
- note added: "10V CHARGE PUMP"
- note added: "POWER SUPPLY"
- note added: "SOFT SWITCH"
- moved on the sheet: BT+, BT-, D8, OFF, OFFSW, ON, PWR, PWRCTL, R28, R29, R30
